Commit message: working iggy simulation using the jackal for visualization

File: urdf/iggy_minimal.urdf.xacro (robot description, xacro)
@@ -1,171 +1,180 @@
 <?xml version="1.0"?>
-<robot name="jackal" xmlns:xacro="http://www.ros.org/wiki/xacro">
-  <xacro:property name="PI" value="3.1415926535897931" />
-  <xacro:property name="wheelbase" value="0.262" /> <!-- TODO UPDATE -->
-  <xacro:property name="track" value="0.37559" /> <!-- TODO UPDATE -->
-  <xacro:property name="wheel_vertical_offset" value="0.0345" /> <!-- TODO UPDATE -->
-  <xacro:property name="footprint_vertical_offset" value="-0.0655" /> <!-- TODO UPDATE -->
-  <xacro:property name="wheel_radius" value="0.098" /> <!-- TODO UPDATE -->
-  <xacro:property name="wheel_width" value="0.040" /> <!-- TODO UPDATE -->
-  <xacro:property name="chassis_length" value="0.914" />
-  <xacro:property name="chassis_width" value="0.609" />
-  <xacro:property name="chassis_height" value="0.184" /> <!-- TODO UPDATE -->
-  <xacro:property name="dummy_inertia" value="1e-09"/>
-  <xacro:property name="mount_spacing" value="0.120" /> <!-- TODO UPDATE -->
-  <material name="dark_grey"><color rgba="0.2 0.2 0.2 1.0" /></material>
-  <material name="light_grey"><color rgba="0.4 0.4 0.4 1.0" /></material>
-  <material name="yellow"><color rgba="0.8 0.8 0.0 1.0" /></material>
-  <material name="black"><color rgba="0.15 0.15 0.15 1.0" /></material>
-  <xacro:macro name="wheel" params="prefix *joint_pose">
-    <link name="${prefix}_wheel_link">
-      <visual>
-        <origin xyz="0 0 0" rpy="${PI/2} 0 0"/>
-        <geometry>
-          <mesh filename="package://iggy_description/meshes/jackal-wheel.stl"/>
-        </geometry>
-        <material name="black" />
-      </visual>
-      <collision>
-        <origin xyz="0 0 0" rpy="${PI/2} 0 0"/>
-        <geometry>
-          <cylinder radius="${wheel_radius}" length="${wheel_width}"/>
-        </geometry>
-      </collision>
-      <inertial>
-        <origin xyz="0 0 0" rpy="0 0 0"/>
-        <mass value="0.477"/>
-        <inertia
-          ixx="0.0013" ixy="0" ixz="0"
-          iyy="0.0024" iyz="0"
-          izz="0.0013"/>
-      </inertial>
+<robot name="iggy" xmlns:xacro="http://www.ros.org/wiki/xacro" xmlns:controller="http://playerstage.sourceforge.net/gazebo/xmlschema/#controller">
+    <xacro:property name="PI" value="3.1415926535897931" />
+    <xacro:property name="wheelbase" value="0.262" />    <!-- TODO UPDATE -->
+    <xacro:property name="track" value="0.37559" />    <!-- TODO UPDATE -->
+    <xacro:property name="wheel_vertical_offset" value="0.0345" />    <!-- TODO UPDATE -->
+    <xacro:property name="footprint_vertical_offset" value="-0.0655" />    <!-- TODO UPDATE -->
+    <xacro:property name="wheel_radius" value="0.098" />    <!-- TODO UPDATE -->
+    <xacro:property name="wheel_width" value="0.040" />    <!-- TODO UPDATE -->
+    <xacro:property name="chassis_length" value="0.914" />    <!-- TODO UPDATE -->
+    <xacro:property name="chassis_width" value="0.609" />    <!-- TODO UPDATE -->
+    <xacro:property name="chassis_height" value="0.184" />    <!-- TODO UPDATE -->
+    <xacro:property name="dummy_inertia" value="1e-09" />    <!-- TODO UPDATE -->
+    <xacro:property name="mount_spacing" value="0.120" />    <!-- TODO UPDATE -->
+    <material name="dark_grey">
+        <color rgba="0.2 0.2 0.2 1.0" />
+    </material>
+    <material name="light_grey">
+        <color rgba="0.4 0.4 0.4 1.0" />
+    </material>
+    <material name="yellow">
+        <color rgba="0.8 0.8 0.0 1.0" />
+    </material>
+    <material name="black">
+        <color rgba="0.15 0.15 0.15 1.0" />
+    </material>
+    <xacro:macro name="wheel" params="prefix *joint_pose">
+        <link name="${prefix}_wheel_link">
+            <visual>
+                <origin xyz="0 0 0" rpy="${PI/2} 0 0" />
+                <geometry>
+                    <mesh filename="package://iggy_description/meshes/jackal-wheel.stl" />
+                </geometry>
+                <material name="black" />
+            </visual>
+            <collision>
+                <origin xyz="0 0 0" rpy="${PI/2} 0 0" />
+                <geometry>
+                    <cylinder radius="${wheel_radius}" length="${wheel_width}" />
+                </geometry>
+            </collision>
+            <inertial>
+                <origin xyz="0 0 0" rpy="0 0 0" />
+                <mass value="0.477" />
+                <inertia ixx="0.0013" ixy="0" ixz="0" iyy="0.0024" iyz="0" izz="0.0013" />
+            </inertial>
+        </link>
+        <gazebo reference="${prefix}_wheel_link">
+            <material>Gazebo/DarkGrey</material>
+        </gazebo>
+        <joint name="${prefix}_wheel" type="continuous">
+            <parent link="chassis_link" />
+            <child link="${prefix}_wheel_link" />
+            <xacro:insert_block name="joint_pose" />
+            <axis xyz="0 1 0" />
+        </joint>
+        <!-- Create a transmission for each wheel -->
+        <transmission name="${prefix}_wheel_trans">
+            <type>transmission_interface/SimpleTransmission</type>
+            <joint name="${prefix}_wheel">
+                <hardwareInterface>VelocityJointInterface</hardwareInterface>
+            </joint>
+            <actuator name="${prefix}_actuator">
+                <mechanicalReduction>1</mechanicalReduction>
+            </actuator>
+        </transmission>
+    </xacro:macro>
+    <!-- TODO Create Caster to replace front wheels  -->
+    <xacro:wheel prefix="front_left">
+        <origin xyz="${wheelbase/2} ${track/2} ${wheel_vertical_offset}" rpy="0 0 0" />
+    </xacro:wheel>
+    <xacro:wheel prefix="front_right">
+        <origin xyz="${wheelbase/2} ${-track/2} ${wheel_vertical_offset}" rpy="0 0 0" />
+    </xacro:wheel>
+    <xacro:wheel prefix="rear_left">
+        <origin xyz="${-wheelbase/2} ${track/2} ${wheel_vertical_offset}" rpy="0 0 0" />
+    </xacro:wheel>
+    <xacro:wheel prefix="rear_right">
+        <origin xyz="${-wheelbase/2} ${-track/2} ${wheel_vertical_offset}" rpy="0 0 0" />
+    </xacro:wheel>
+    <link name="base_link"></link>
+    <joint name="base_link_joint" type="fixed">
+        <origin xyz="0 0 0" rpy="0 0 0" />
+        <parent link="base_link" />
+        <child link="chassis_link" />
+    </joint>
+    <link name="chassis_link">
+        <visual>
+            <origin xyz="0 0 ${footprint_vertical_offset}" rpy="${PI/2} 0 ${PI/2}" />
+            <geometry>
+                <mesh filename="package://iggy_description/meshes/jackal-base.stl" />
+            </geometry>
+            <material name="dark_grey" />
+        </visual>
+        <collision>
+            <origin xyz="0 0 ${chassis_height/2}" />
+            <geometry>
+                <box size="${chassis_length} ${chassis_width} ${chassis_height}" />
+            </geometry>
+        </collision>
+        <inertial>
+            <!-- Center of mass -->
+            <origin xyz="0.012  0.002 0.067" rpy="0 0 0" />
+            <mass value="16.523" />
+            <!-- Moments of inertia: ( chassis without wheels ) -->
+            <inertia ixx="0.3136" ixy="-0.0008" ixz="0.0164" iyy="0.3922" iyz="-0.0009" izz="0.4485" />
+        </inertial>
     </link>
-    <gazebo reference="${prefix}_wheel_link">
-      <material>Gazebo/DarkGrey</material>
-    </gazebo>
-    <joint name="${prefix}_wheel" type="continuous">
-      <parent link="chassis_link"/>
-      <child link="${prefix}_wheel_link" />
-      <xacro:insert_block name="joint_pose" />
-      <axis xyz="0 1 0" />
+    <!-- TODO IGGY does not have fenders. What to do with this?? -->
+    <link name="fenders_link">
+        <visual>
+            <origin xyz="0 0 ${footprint_vertical_offset}" rpy="${PI/2} 0 ${PI/2}" />
+            <geometry>
+                <mesh filename="package://iggy_description/meshes/jackal-fenders.stl" />
+            </geometry>
+            <material name="yellow" />
+        </visual>
+    </link>
+    <joint name="fenders_joint" type="fixed">
+        <parent link="chassis_link" />
+        <child link="fenders_link" />
     </joint>
-    <!-- Create a transmission for each wheel -->
-    <transmission name="${prefix}_wheel_trans">
-      <type>transmission_interface/SimpleTransmission</type>
-      <joint name="${prefix}_wheel">
-        <hardwareInterface>VelocityJointInterface</hardwareInterface>
-      </joint>
-      <actuator name="${prefix}_actuator">
-        <mechanicalReduction>1</mechanicalReduction>
-      </actuator>
-    </transmission>
-  </xacro:macro>
-<!-- TODO Create Caster to replace front wheels  -->
-  <xacro:wheel prefix="front_left">
-    <origin xyz="${wheelbase/2} ${track/2} ${wheel_vertical_offset}" rpy="0 0 0" />
-  </xacro:wheel>
-  <xacro:wheel prefix="front_right">
-    <origin xyz="${wheelbase/2} ${-track/2} ${wheel_vertical_offset}" rpy="0 0 0" />
-  </xacro:wheel>
-  <xacro:wheel prefix="rear_left">
-    <origin xyz="${-wheelbase/2} ${track/2} ${wheel_vertical_offset}" rpy="0 0 0" />
-  </xacro:wheel>
-  <xacro:wheel prefix="rear_right">
-    <origin xyz="${-wheelbase/2} ${-track/2} ${wheel_vertical_offset}" rpy="0 0 0" />
-  </xacro:wheel>
-  <link name="base_link"></link>
-  <joint name="base_link_joint" type="fixed">
-    <origin xyz="0 0 0" rpy="0 0 0" />
-    <parent link="base_link"/>
-    <child link="chassis_link" />
-  </joint>
-  <link name="chassis_link">
-    <visual>
-      <origin xyz="0 0 ${footprint_vertical_offset}" rpy="${PI/2} 0 ${PI/2}"/>
-      <geometry>
-        <mesh filename="package://iggy_description/meshes/jackal-base.stl"/>
-      </geometry>
-      <material name="dark_grey" />
-    </visual>
-    <collision>
-      <origin xyz="0 0 ${chassis_height/2}"/>
-      <geometry>
-        <box size="${chassis_length} ${chassis_width} ${chassis_height}"/>
-      </geometry>
-    </collision>
-    <inertial>
-      <!-- Center of mass -->
-      <origin xyz="0.012  0.002 0.067" rpy="0 0 0"/>
-      <mass value="16.523"/>
-      <!-- Moments of inertia: ( chassis without wheels ) -->
-      <inertia
-        ixx="0.3136" ixy="-0.0008" ixz="0.0164"
-        iyy="0.3922" iyz="-0.0009"
-        izz="0.4485"/>
-      </inertial>
-  </link>
-  <!-- TODO IGGY does not have fenders. What to do with this?? -->
-  <link name="fenders_link">
-    <visual>
-      <origin xyz="0 0 ${footprint_vertical_offset}" rpy="${PI/2} 0 ${PI/2}"/>
-      <geometry>
-        <mesh filename="package://iggy_description/meshes/jackal-fenders.stl"/>
-      </geometry>
-      <material name="yellow" />
-    </visual>
-  </link>
-  <joint name="fenders_joint" type="fixed">
-    <parent link="chassis_link" />
-    <child link="fenders_link" />
-  </joint>
-  <!-- TODO: Make this internal_imu_link or something, and use a mixed-in xacro
+    <!-- TODO: Make this internal_imu_link or something, and use a mixed-in xacro
        to supply the joint between it and imu_link. This is important so that imu_link
        always points to the "active" IMU. When an upgrade IMU is connected, the
        internal_imu_link should remain, but imu_link should point to the upgrade one. -->
-  <link name="imu_link">
-    <inertial>
-      <mass value="0.001"/>
-      <origin xyz="0 0 0" rpy="0 0 0"/>
-      <inertia ixx="${dummy_inertia}" ixy="0.0" ixz="0.0" iyy="${dummy_inertia}" iyz="0.0" izz="${dummy_inertia}"/>
-    </inertial>
-  </link>
-  <joint name="imu_joint" type="fixed">
-    <parent link="chassis_link" />
-    <child link="imu_link" />
-  </joint>
-  <!-- TODO: Same note as applies to imu_link -->
-  <link name="navsat_link">
-    <visual>
-      <geometry>
-        <cylinder radius="0.026" length="0.016" />
-      </geometry>
-      <origin xyz="0 0 0.008" />
-      <material name="black" />
-    </visual>
-  </link>
-  <joint name="navsat_joint" type="fixed">
-    <parent link="chassis_link" />
-    <child link="navsat_link" />
-    <origin xyz="-0.180 0.126 0.1815" />
-  </joint>
-  <link name="mid_mount"></link>
-  <joint name="mid_mount_joint" type="fixed">
-    <parent link="chassis_link" />
-    <child link="mid_mount" />
-    <origin xyz="0 0 ${chassis_height}" />
-  </joint>
-  <link name="rear_mount"></link>
-  <joint name="rear_mount_joint" type="fixed">
-    <parent link="mid_mount" />
-    <child link="rear_mount" />
-    <origin xyz="${-mount_spacing} 0 0" />
-  </joint>
-  <link name="front_mount"></link>
-  <joint name="front_mount_joint" type="fixed">
-    <parent link="mid_mount" />
-    <child link="front_mount" />
-    <origin xyz="${mount_spacing} 0 0" />
-  </joint>
-  <!-- Bring in simulation data for Gazebo. -->
-  <xacro:include filename="iggy.gazebo" />
+    <link name="imu_link">
+        <inertial>
+            <mass value="0.001" />
+            <origin xyz="0 0 0" rpy="0 0 0" />
+            <inertia ixx="${dummy_inertia}" ixy="0.0" ixz="0.0" iyy="${dummy_inertia}" iyz="0.0" izz="${dummy_inertia}" />
+        </inertial>
+    </link>
+    <joint name="imu_joint" type="fixed">
+        <parent link="chassis_link" />
+        <child link="imu_link" />
+    </joint>
+    <!-- TODO: Same note as applies to imu_link -->
+    <link name="navsat_link">
+        <visual>
+            <geometry>
+                <cylinder radius="0.026" length="0.016" />
+            </geometry>
+            <origin xyz="0 0 0.008" />
+            <material name="black" />
+        </visual>
+    </link>
+    <joint name="navsat_joint" type="fixed">
+        <parent link="chassis_link" />
+        <child link="navsat_link" />
+        <origin xyz="-0.180 0.126 0.1815" />
+    </joint>
+    <link name="mid_mount"></link>
+    <joint name="mid_mount_joint" type="fixed">
+        <parent link="chassis_link" />
+        <child link="mid_mount" />
+        <origin xyz="0 0 ${chassis_height}" />
+    </joint>
+    <link name="rear_mount"></link>
+    <joint name="rear_mount_joint" type="fixed">
+        <parent link="mid_mount" />
+        <child link="rear_mount" />
+        <origin xyz="${-mount_spacing} 0 0" />
+    </joint>
+    <link name="front_mount"></link>
+    <joint name="front_mount_joint" type="fixed">
+        <parent link="mid_mount" />
+        <child link="front_mount" />
+        <origin xyz="${mount_spacing} 0 0" />
+    </joint>
+    <!-- Bring in simulation data for Gazebo. -->
+    <xacro:include filename="iggy.gazebo" />
 </robot>
+<!-- Some test code used in developing solution ============
+rosrun xacro xacro.py -o iggy_minimal.urdf `rospack find iggy_description`/urdf/iggy_minimal.urdf.xacro
+check_urdf iggy_minimal.urdf
+urdf_to_graphiz iggy_minimal.urdf
+evince iggy_minimal.pdf
+rostopic pub -r 10 /iggy/cmd_vel geometry_msgs/Twist  '{linear:  {x: 0.1, y: 0.0, z: 0.0}, angular: {x: 0.0,y: 0.0,z: 0.0}}'
+================= -->

Commit message: some progress on adding casters

File: urdf/iggy_minimal.urdf.xacro (robot description, xacro)
@@ -1,4 +1,24 @@
 <?xml version="1.0"?>
 <robot name="iggy" xmlns:xacro="http://www.ros.org/wiki/xacro" xmlns:controller="http://playerstage.sourceforge.net/gazebo/xmlschema/#controller">
+  <!-- PROPERTY LIST -->
+  <!--All units in m-kg-s-radians unit system -->
+  <property name="M_PI" value="3.1415926535897931" />
+  <property name="M_PI_2" value="1.570796327" />
+  <property name="DEG_TO_RAD" value="0.017453293" />
+  <!-- Main body radius and height -->
+  <!-- Main Body Cylinder base   -->
+  <property name="base_height" value="0.02" />
+  <property name="base_radius" value="0.15" />
+  <property name="base_mass" value="5" /> <!-- in kg-->
+  <!-- caster wheel radius and height -->
+  <!-- caster wheel mass -->
+  <property name="caster_f_height" value="0.04" />
+  <property name="caster_f_radius" value="0.025" />
+  <property name="caster_f_mass" value="0.5" /> <!-- in kg-->
+  <!-- caster wheel radius and height -->
+  <!-- caster wheel mass -->
+  <property name="caster_b_height" value="0.04" />
+  <property name="caster_b_radius" value="0.025" />
+  <property name="caster_b_mass" value="0.5" /> <!-- in kg-->
     <xacro:property name="PI" value="3.1415926535897931" />
     <xacro:property name="wheelbase" value="0.262" />    <!-- TODO UPDATE -->
@@ -67,7 +87,4 @@
     </xacro:macro>
     <!-- TODO Create Caster to replace front wheels  -->
-    <xacro:wheel prefix="front_left">
-        <origin xyz="${wheelbase/2} ${track/2} ${wheel_vertical_offset}" rpy="0 0 0" />
-    </xacro:wheel>
     <xacro:wheel prefix="front_right">
         <origin xyz="${wheelbase/2} ${-track/2} ${wheel_vertical_offset}" rpy="0 0 0" />
