Commit message: added test.urdf

File: urdf/iggy_minimal.urdf(2).xacro (robot description, xacro)
@@ -14,5 +14,5 @@
   <!-- caster wheel mass -->
   <property name="caster_f_height" value="0.04" />
-  <property name="caster_f_radius" value="0.098" />
+  <property name="caster_f_radius" value="0.025" />
   <property name="caster_f_mass" value="0.5" /> <!-- in kg-->
   <!-- caster wheel radius and height -->
@@ -90,68 +90,69 @@
     </xacro:macro>
     <!-- TODO Create Caster to replace front wheels  -->
-    <!--<xacro:wheel prefix="front_right">
-        <origin xyz="${wheelbase/2} ${track/2} ${wheel_vertical_offset}" rpy="0 0 0" />
-    </xacro:wheel> -->
-    <link name="caster_left_link">
+    <!--Caster front  -->
+    <link name="caster_front_right">
     <visual>
-      <origin rpy="1.57079632679 0 0" xyz="0 0.02 0"/>
+      <origin xyz="${wheelbase/2} ${-track/2} ${wheel_vertical_offset}" rpy="0 0 0" />
       <geometry>
-         <mesh filename="package://iggy_description/meshes/jackal-wheel.stl" />
+	<sphere radius="${caster_f_radius}" />
       </geometry>
-      <material name="Black"/>
+      <material name="Black" />
     </visual>
-    <collision>
-      <origin rpy="1.57079632679 0 0 " xyz="0 0 0"/>
-      <geometry>
-        <cylinder length="0.02" radius="0.04"/>
-      </geometry>
-</collision>
-    <inertial>
-      <mass value="0.5"/>
-      <origin xyz="0 0 0"/>
-      <inertia ixx="0.001" ixy="0.0" ixz="0.0" iyy="0.001" iyz="0.0" izz="0.001"/>
-    </inertial>
-  </link>
-    <gazebo reference="caster_left_link">
+      <collision>
+        <geometry>
+	<sphere radius="${caster_f_radius}" />
+        </geometry>
+      <origin xyz="0 0.02 0" rpy="${M_PI/2} 0 0" />
+      </collision>
+      <inertial>
+        <mass value="${caster_f_mass}" />
+        <origin xyz="0 0 0" />
+        <inertia ixx="0.001" ixy="0.0" ixz="0.0"
+                 iyy="0.001" iyz="0.0"
+                 izz="0.001" />
+      </inertial>
+    </link>
+ <joint name="caster_front_joint" type="fixed">
+      <parent link="base_link"/>
+      <child link="caster_front_link"/>
+      <origin xyz="0.115 0.0 0.007" rpy="${-M_PI/2} 0 0"/>
+    </joint>
+  <gazebo reference="caster_front_link">
     <turnGravityOff>false</turnGravityOff>
   </gazebo>
-  <joint name="caster_left_joint" type="fixed">
-  <dynamics damping="0.0" friction="0.0"/>
-    <parent link="base_link"/>
-    <child link="caster_left_link"/>
-    <origin rpy="0 0 0" xyz="${wheelbase/2} ${track/2} ${wheel_vertical_offset}"/>
-</joint>
-   <!-- <xacro:wheel prefix="front_left">
-        <origin xyz="${wheelbase/2} ${-track/2} ${wheel_vertical_offset}" rpy="0 0 0" />
-    </xacro:wheel> -->
-<link name="caster_right_link">
+    <!--<xacro:wheel prefix="front_right">
+        <origin xyz="${wheelbase/2} ${-track/2} ${wheel_vertical_offset}" rpy="0 0 0" /> -->
+    <!--Caster front  -->
+    <link name="caster_front_link">
     <visual>
-      <origin rpy="1.57079632679 0 0" xyz="0 0.02 0"/>
+      <origin xyz="0 0.02 0" rpy="${M_PI/2} 0 0" />
       <geometry>
-         <mesh filename="package://iggy_description/meshes/jackal-wheel.stl" />
+	<sphere radius="${caster_f_radius}" />
       </geometry>
-      <material name="Black"/>
+      <material name="Black" />
     </visual>
-    <collision>
-      <origin rpy="1.57079632679 0 0 " xyz="0 0 0"/>
-      <geometry>
-        <cylinder length="0.02" radius="0.04"/>
-      </geometry>
-</collision>
-    <inertial>
-      <mass value="0.5"/>
-      <origin xyz="0 0 0"/>
-      <inertia ixx="0.001" ixy="0.0" ixz="0.0" iyy="0.001" iyz="0.0" izz="0.001"/>
-    </inertial>
-  </link>
-    <gazebo reference="caster_right_link">
+      <collision>
+        <geometry>
+	<sphere radius="${caster_f_radius}" />
+        </geometry>
+      <origin xyz="0 0.02 0" rpy="${M_PI/2} 0 0" />
+      </collision>
+      <inertial>
+        <mass value="${caster_f_mass}" />
+        <origin xyz="0 0 0" />
+        <inertia ixx="0.001" ixy="0.0" ixz="0.0"
+                 iyy="0.001" iyz="0.0"
+                 izz="0.001" />
+      </inertial>
+    </link>
+ <joint name="caster_front_joint" type="fixed">
+      <parent link="base_link"/>
+      <child link="caster_front_link"/>
+      <origin xyz="0.115 0.0 0.007" rpy="${-M_PI/2} 0 0"/>
+    </joint>
+  <gazebo reference="caster_front_link">
     <turnGravityOff>false</turnGravityOff>
   </gazebo>
-  <joint name="caster_front_joint" type="fixed">
-  <dynamics damping="0.0" friction="0.0"/>
-    <parent link="base_link"/>
-    <child link="caster_right_link"/>
-    <origin rpy="0 0 0" xyz="${wheelbase/2} ${-track/2} ${wheel_vertical_offset}"/>
-</joint>
+    </xacro:wheel>
     <xacro:wheel prefix="rear_left">
         <origin xyz="${-wheelbase/2} ${track/2} ${wheel_vertical_offset}" rpy="0 0 0" />
