Commit message: still not working wheels not properly placed

File: urdf/test2.urdf (robot description, URDF)
Before this commit: robot differential_wheeled_robot, 9 links, 8 joints
Links:
- removed link back_wheel_base
- removed link caster_back_link
- removed link caster_front_link
- removed link front_wheel_base
- added link caster_link_left, mass 0.5; collision sphere radius=0.08; visual sphere radius=0.025
- added link caster_link_right, mass 10; collision sphere radius=0.08; visual sphere radius=0.025
- added link middle_link_left, mass 5; collision box size=.02 .01 .02; visual box size=.1 .1 .01
- added link middle_link_right, mass 10; collision box size=.02 .01 .02; visual box size=.1 .1 .01
- added link weight, mass 50; collision box size=.02 .01 .02; visual box size=.1 .1 .01
- link base_link: mass 50 -> 5
- link front_left_wheel: geometry collision cylinder length=0.02 radius=0.04; visual cylinder length=0.02 radius=0.04
- link front_right_wheel: geometry collision cylinder length=0.02 radius=0.04; visual cylinder length=0.02 radius=0.04
Joints:
- removed joint back_wheel_base_to_base_link
- removed joint caster_back_joint
- removed joint caster_front_joint
- removed joint front_wheel_base_to_base_link
- added joint top_joint_left: type revolute, parent base_link, child middle_link_left, origin xyz=.1 .15 -.18 rpy=0 0 0, axis 0 0 1, limit lower=0.0 upper=0.548 effort=1000.0 velocity=0.5
- added joint top_joint_right: type revolute, parent base_link, child middle_link_right, origin xyz=.1 -.15 -.18 rpy=0 0 0, axis 0 0 1, limit lower=0.0 upper=0.548 effort=1000.0 velocity=0.5
- added joint wheel_joint_left: type fixed, parent middle_link_left, child caster_link_left, origin xyz=0 0 0 rpy=-1.57079632679 0 0
- added joint wheel_joint_right: type fixed, parent middle_link_right, child caster_link_right, origin xyz=0 0 0 rpy=-1.57079632679 0 0
- added joint wight_joint: type fixed, parent base_link, child weight, origin xyz=.10 .20 .30 rpy=-1.57079632679 0 0
- joint front_left_wheel_joint: origin xyz=0 .15 -.18 rpy=0 0 0 -> xyz=-.1 -.15 -.18 rpy=0 0 0; parent back_wheel_base -> base_link
- joint front_right_wheel_joint: origin xyz=0 -.15 -.18 rpy=0 0 0 -> xyz=-.1 .15 -.18 rpy=0 0 0; parent back_wheel_base -> base_link
